File: Hardware/led-matrix-v4/led-matrix-v4.kicad_pcb (KiCad board)
At the start: 4 copper layers, 245 x 209 mm, 517 parts, among them J1 Conn_01x04_Socket, U1 SN74AHCT125DR

Commit message: replaced mounting holes, filled power layers
Parts:
- added REF**: MountingHole_2.2mm_M2_DIN965_Pad, MountingHole:MountingHole_2.2mm_M2_DIN965_Pad, F.Cu at (44.0, 45.0)
- added REF**: MountingHole_2.2mm_M2_DIN965_Pad, MountingHole:MountingHole_2.2mm_M2_DIN965_Pad, F.Cu at (44.0, 249.0)
- added REF**: MountingHole_2.2mm_M2_DIN965_Pad, MountingHole:MountingHole_2.2mm_M2_DIN965_Pad, F.Cu at (281.0, 45.0)
- added REF**: MountingHole_2.2mm_M2_DIN965_Pad, MountingHole:MountingHole_2.2mm_M2_DIN965_Pad, F.Cu at (281.0, 249.0)
Routing:
- net GND: track 62.2 -> 7.65 mm
- net VDD: track 21.1 -> 9.21 mm
Other:
- board size 245 x 209 mm -> 245 x 212 mm
Changed lines of the file:
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@@
     )
   )
+  (footprint "MountingHole:MountingHole_2.2mm_M2_DIN965_Pad" (layer "F.Cu")
+    (at 44 45)
+    (descr "Mounting Hole 2.2mm, M2, DIN965")
+    (tags "mounting hole 2.2mm m2 din965")
+    (attr exclude_from_pos_files exclude_from_bom)
+    (fp_text reference "REF**" (at 0 -2.9) (layer "F.SilkS") hide
+        (effects (font (size 1 1) (thickness 0.15)))
+    )
+    (fp_text value "MountingHole_2.2mm_M2_DIN965_Pad" (at 0 2.9) (layer "F.Fab") hide
+        (effects (font (size 1 1) (thickness 0.15)))
+    )
+    (fp_text user "${REFERENCE}" (at 0 0) (layer "F.Fab")
+        (effects (font (size 1 1) (thickness 0.15)))
+    )
+    (fp_circle (center 0 0) (end 1.9 0)
+      (stroke (width 0.15) (type solid)) (fill none) (layer "Cmts.User"))
+    (fp_circle (center 0 0) (end 2.15 0)
+      (stroke (width 0.05) (type solid)) (fill none) (layer "F.CrtYd"))
+    (pad "1" thru_hole circle (at 0 0) (size 3.8 3.8) (drill 2.2) (layers "*.Cu" "*.Mask")
+      (net 2 "GND"))
+  )
   (footprint "LED_SMD:LED_WS2812B_PLCC4_5.0x5.0mm_P3.2mm" (layer "F.Cu")
     (at 159.65 114)
@@
     )
   )
+  (footprint "MountingHole:MountingHole_2.2mm_M2_DIN965_Pad" (layer "F.Cu")
+    (at 44 249)
+    (descr "Mounting Hole 2.2mm, M2, DIN965")
+    (tags "mounting hole 2.2mm m2 din965")
+    (attr exclude_from_pos_files exclude_from_bom)
+    (fp_text reference "REF**" (at 0 -2.9) (layer "F.SilkS") hide
+        (effects (font (size 1 1) (thickness 0.15)))
+    )
+    (fp_text value "MountingHole_2.2mm_M2_DIN965_Pad" (at 0 2.9) (layer "F.Fab") hide
+        (effects (font (size 1 1) (thickness 0.15)))
+    )
+    (fp_text user "${REFERENCE}" (at 0 0) (layer "F.Fab")
+        (effects (font (size 1 1) (thickness 0.15)))
+    )
+    (fp_circle (center 0 0) (end 1.9 0)
+      (stroke (width 0.15) (type solid)) (fill none) (layer "Cmts.User"))
+    (fp_circle (center 0 0) (end 2.15 0)
+      (stroke (width 0.05) (type solid)) (fill none) (layer "F.CrtYd"))
+    (pad "1" thru_hole circle (at 0 0) (size 3.8 3.8) (drill 2.2) (layers "*.Cu" "*.Mask")
+      (net 2 "GND"))
+  )
   (footprint "LED_SMD:LED_WS2812B_PLCC4_5.0x5.0mm_P3.2mm" (layer "F.Cu")
     (at 134.25 101.3)
@@
     )
   )
+  (footprint "MountingHole:MountingHole_2.2mm_M2_DIN965_Pad" (layer "F.Cu")
+    (at 281 45)
+    (descr "Mounting Hole 2.2mm, M2, DIN965")
+    (tags "mounting hole 2.2mm m2 din965")
+    (attr exclude_from_pos_files exclude_from_bom)
+    (fp_text reference "REF**" (at 0 -2.9) (layer "F.SilkS") hide
+        (effects (font (size 1 1) (thickness 0.15)))
+    )
+    (fp_text value "MountingHole_2.2mm_M2_DIN965_Pad" (at 0 2.9) (layer "F.Fab") hide
+        (effects (font (size 1 1) (thickness 0.15)))
+    )
+    (fp_text user "${REFERENCE}" (at 0 0) (layer "F.Fab")
+        (effects (font (size 1 1) (thickness 0.15)))
+    )
+    (fp_circle (center 0 0) (end 1.9 0)
+      (stroke (width 0.15) (type solid)) (fill none) (layer "Cmts.User"))
+    (fp_circle (center 0 0) (end 2.15 0)
+      (stroke (width 0.05) (type solid)) (fill none) (layer "F.CrtYd"))
+    (pad "1" thru_hole circle (at 0 0) (size 3.8 3.8) (drill 2.2) (layers "*.Cu" "*.Mask")
+      (net 2 "GND"))
+  )
   (footprint "LED_SMD:LED_WS2812B_PLCC4_5.0x5.0mm_P3.2mm" (layer "F.Cu")
     (at 172.35 228.3)
@@
     )
   )
+  (footprint "MountingHole:MountingHole_2.2mm_M2_DIN965_Pad" (layer "F.Cu")
+    (at 281 249)
+    (descr "Mounting Hole 2.2mm, M2, DIN965")
+    (tags "mounting hole 2.2mm m2 din965")
+    (attr exclude_from_pos_files exclude_from_bom)
+    (fp_text reference "REF**" (at 0 -2.9) (layer "F.SilkS") hide
+        (effects (font (size 1 1) (thickness 0.15)))
+    )
+    (fp_text value "MountingHole_2.2mm_M2_DIN965_Pad" (at 0 2.9) (layer "F.Fab") hide
+        (effects (font (size 1 1) (thickness 0.15)))
+    )
+    (fp_text user "${REFERENCE}" (at 0 0) (layer "F.Fab")
+        (effects (font (size 1 1) (thickness 0.15)))
+    )
+    (fp_circle (center 0 0) (end 1.9 0)
+      (stroke (width 0.15) (type solid)) (fill none) (layer "Cmts.User"))
+    (fp_circle (center 0 0) (end 2.15 0)
+      (stroke (width 0.05) (type solid)) (fill none) (layer "F.CrtYd"))
+    (pad "1" thru_hole circle (at 0 0) (size 3.8 3.8) (drill 2.2) (layers "*.Cu" "*.Mask")
+      (net 2 "GND"))
+  )
   (footprint "LED_SMD:LED_WS2812B_PLCC4_5.0x5.0mm_P3.2mm" (layer "F.Cu")
     (at 96.15 63.2)
@@
     )
   )
-  (gr_line (start 280.971573 44) (end 44 44)
+  (gr_line (start 40 45) (end 40 249)
     (stroke (width 0.1) (type default)) (layer "Edge.Cuts"))
-  (gr_line (start 40 48) (end 40 249)
-    (stroke (width 0.1) (type default)) (layer "Edge.Cuts"))
-  (gr_circle (center 44 249) (end 42 249)
-    (stroke (width 0.1) (type default)) (fill none) (layer "Edge.Cuts"))
-  (gr_arc (start 280.971573 44) (mid 283.8 45.171573) (end 284.971573 48)
-    (stroke (width 0.1) (type default)) (layer "Edge.Cuts"))
-  (gr_circle (center 280.971573 48) (end 281 46)
-    (stroke (width 0.1) (type default)) (fill none) (layer "Edge.Cuts"))
   (gr_arc (start 284.971573 249) (mid 283.8 251.828427) (end 280.971573 253)
     (stroke (width 0.1) (type default)) (layer "Edge.Cuts"))
   (gr_line (start 44 253) (end 280.971573 253)
     (stroke (width 0.1) (type default)) (layer "Edge.Cuts"))
-  (gr_circle (center 280.971573 249) (end 281 251)
-    (stroke (width 0.1) (type default)) (fill none) (layer "Edge.Cuts"))
-  (gr_line (start 284.971573 249) (end 284.971573 48)
+  (gr_line (start 284.971573 249) (end 284.971573 45)
     (stroke (width 0.1) (type default)) (layer "Edge.Cuts"))
   (gr_arc (start 44 253) (mid 41.171573 251.828427) (end 40 249)
     (stroke (width 0.1) (type default)) (layer "Edge.Cuts"))
-  (gr_arc (start 40 48) (mid 41.171573 45.171573) (end 44 44)
+  (gr_arc (start 280.971573 41) (mid 283.8 42.171573) (end 284.971573 45)
+    (stroke (width 0.1) (type default)) (layer "Edge.Cuts"))
+  (gr_line (start 280.971573 41) (end 44 41)
+    (stroke (width 0.1) (type default)) (layer "Edge.Cuts"))
+  (gr_arc (start 40 45) (mid 41.171573 42.171573) (end 44 41)
     (stroke (width 0.1) (type default)) (layer "Edge.Cuts"))
-  (gr_circle (center 44 48) (end 42 48)
-    (stroke (width 0.1) (type default)) (fill none) (layer "Edge.Cuts"))
   (gr_text "LED MATRIX v4\nUCCS ECE4898 FALL 2023\nDesigned by Eleanor Taylor" (at 76.4 239.1 90) (layer "F.SilkS")
     (effects (font (size 1 1) (thickness 0.15)) (justify left bottom))
@@
   (via blind (at 144.5 226.6) (size 0.8) (drill 0.4) (layers "F.Cu" "In1.Cu") (net 1))
   (segment (start 66.1 123.6512) (end 66.1 115.525) (width 0.25) (layer "In1.Cu") (net 1))
-  (segment (start 66.8638 124.415) (end 78.785 124.415) (width 0.25) (layer "In1.Cu") (net 1))
   (segment (start 66.8638 124.415) (end 66.1 123.6512) (width 0.25) (layer "In1.Cu") (net 1))
-  (segment (start 78.785 124.415) (end 78.8 124.4) (width 0.25) (layer "In1.Cu") (net 1))
   (via blind (at 84.4 183.8) (size 0.8) (drill 0.4) (layers "In1.Cu" "B.Cu") (net 1))
   (via blind (at 97.1 94.9) (size 0.8) (drill 0.4) (layers "In1.Cu" "B.Cu") (net 1))
@@
   (via blind (at 187.5 179.1) (size 0.8) (drill 0.4) (layers "F.Cu" "In2.Cu") (net 2))
   (segment (start 124 52.15) (end 124.15 52.3) (width 0.25) (layer "In2.Cu") (net 2))
-  (segment (start 51.7 118.7) (end 55.1 122.1) (width 0.25) (layer "In2.Cu") (net 2))
-  (segment (start 63.4875 122.125) (end 71 122.125) (width 0.25) (layer "In2.Cu") (net 2))
   (segment (start 149.4 52.15) (end 149.45 52.2) (width 0.25) (layer "In2.Cu") (net 2))
-  (segment (start 64.4 115.525) (end 71 122.125) (width 0.25) (layer "In2.Cu") (net 2))
-  (segment (start 63.4875 122.125) (end 63.4875 130.5426) (width 0.25) (layer "In2.Cu") (net 2))
-  (segment (start 71 122.125) (end 78.775 122.125) (width 0.25) (layer "In2.Cu") (net 2))
-  (segment (start 55.1 122.1) (end 63.4625 122.1) (width 0.25) (layer "In2.Cu") (net 2))
   (segment (start 85.9 52.15) (end 85.95 52.2) (width 0.25) (layer "In2.Cu") (net 2))
+  (segment (start 64.4 121.2125) (end 63.4875 122.125) (width 0.25) (layer "In2.Cu") (net 2))
+  (segment (start 64.4 115.525) (end 64.4 121.2125) (width 0.25) (layer "In2.Cu") (net 2))
   (segment (start 63.4625 122.1) (end 63.4875 122.125) (width 0.25) (layer "In2.Cu") (net 2))
   (segment (start 98.6 52.15) (end 98.75 52.3) (width 0.25) (layer "In2.Cu") (net 2))
-  (segment (start 63.4875 130.5426) (end 61.9362 132.0939) (width 0.25) (layer "In2.Cu") (net 2))
-  (segment (start 78.775 122.125) (end 78.8 122.1) (width 0.25) (layer "In2.Cu") (net 2))
   (segment (start 136.7 52.15) (end 136.75 52.1) (width 0.25) (layer "In2.Cu") (net 2))
-  (segment (start 51.7 118.7) (end 51.7 105.6) (width 0.25) (layer "In2.Cu") (net 2))
   (via blind (at 260.3 234.6) (size 0.8) (drill 0.4) (layers "In2.Cu" "B.Cu") (net 2))
   (via blind (at 82.5 145.7) (size 0.8) (drill 0.4) (layers "In2.Cu" "B.Cu") (net 2))
@@
     (polygon
       (pts
-        (xy 78 47)
-        (xy 278 47)
-        (xy 278 250)
-        (xy 78 250)
+        (xy 40 41)
+        (xy 285 41)
+        (xy 285 253)
+        (xy 40 253)
       )
     )
@@
     (polygon
       (pts
-        (xy 78 47)
-        (xy 278 47)
-        (xy 278 250)
-        (xy 78 250)
+        (xy 40 41)
+        (xy 285 41)
+        (xy 285 253)
+        (xy 40 253)
       )
     )
