File: Hardware/led-matrix-v4/led-matrix-v4.kicad_sch (KiCad schematic)
At the start: 517 parts, among them J1 Conn_01x04_Socket, U1 SN74AHCT125DR

Commit message: fixed dates, etc
Other:
- company: (none) -> UCCS Senior Design Fall 2023
- title: (none) -> LED Matrix
Changed lines of the file:
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@@
 (kicad_sch (version 20230121) (generator eeschema)
   (paper "A1")
+  (title_block
+    (title "LED Matrix")
+    (date "2023-07-19")
+    (rev "4")
+    (company "UCCS Senior Design Fall 2023")
+    (comment 1 "Designed by Eleanor Taylor")
+  )
   (junction (at 417.83 393.7) (diameter 0) (color 0 0 0 0)
   )
