File: Hardware/led-matrix-v2-0/led-matrix-v2-0.kicad_sch (KiCad schematic)
At the start: 517 parts, among them J1 Conn_01x04_Socket, J2 USB_C_Receptacle_PowerOnly_6P, U1 SN74AHCT125DR

Commit message: updated buffer symbol, grounded enables
Connections:
- net GND: now also U1.1 (*1OE), U1.10 (*3OE), U1.13 (*4OE), U1.4 (*2OE)
- no-connect marks 8 -> 4
Other:
- moved on the sheet: J1, J2, R1, R2, U1
