File: Hardware/led-matrix-v2-0/led-matrix-v2-0.kicad_sch (KiCad schematic)
At the start: 517 parts, among them J1 Conn_01x04_Socket, J2 USB_C_Receptacle_PowerOnly_6P, U1 SN74AHCT125DR

Commit message: finished schematics and part selection
Parts:
- added C257: 10u, Capacitor_SMD:C_0805_2012Metric, symbol Device:C
- added C258: 4.7u, Capacitor_SMD:C_0805_2012Metric, symbol Device:C
- added D257: MBR230S1F-7, Diode_SMD:D_SOD-123F, symbol Device:D_Schottky
- added R3: 102k, Resistor_SMD:R_0805_2012Metric, symbol Device:R_US
- added R4: 20k, Resistor_SMD:R_0805_2012Metric, symbol Device:R_US
- added U2: TPS66121, TPS6612x:TPS66121, symbol TPS6612x:TPS66121
Connections:
- net GND: now also C257.2, C258.2, D257.2 (A), R4.2, U2.A3 (GND), U2.A4 (GND), U2.B4 (GND), U2.C4 (GND), U2.D4 (GND), U2.E4 (GND), U2.G4 (VIN)
- net VDD: now also C257.1, D257.1 (K), R3.2, U2.A2 (VBUS), U2.B2 (VBUS), U2.B3 (VBUS), U2.C2 (VBUS), U2.C3 (VBUS), U2.D2 (VBUS), U2.D3 (VBUS), U2.E2 (VBUS), U2.E3 (VBUS), U2.F2 (VBUS), U2.F3 (VBUS), U2.G1 (EN0), U2.G2 (VBUS); no longer U1.14 (VCC)
- new net: C258.1, U2.G3 (VLDO)
- new net: R3.1, R4.1, U2.F4 (OVP)
- new net: U1.14 (VCC), U2.B1 (PPHV), U2.C1 (PPHV), U2.D1 (PPHV), U2.E1 (PPHV), U2.F1 (PPHV)
- no-connect marks 4 -> 5
Other:
- moved on the sheet: J1, R2

Commit message: laid out, routed design
Connections:
- net VDD: now also U1.14 (VCC), U2.B1 (PPHV), U2.C1 (PPHV), U2.D1 (PPHV), U2.E1 (PPHV), U2.F1 (PPHV); no longer C257.1, D257.1 (K), J2.A9 (VBUS), J2.B9 (VBUS), R3.2, U2.A2 (VBUS), U2.B2 (VBUS), U2.B3 (VBUS), U2.C2 (VBUS), U2.C3 (VBUS), U2.D2 (VBUS), U2.D3 (VBUS), U2.E2 (VBUS), U2.E3 (VBUS), U2.F2 (VBUS), U2.F3 (VBUS), U2.G1 (EN0), U2.G2 (VBUS)
- new net: C257.1, D257.1 (K), J2.A9 (VBUS), J2.B9 (VBUS), R3.2, U2.A2 (VBUS), U2.B2 (VBUS), U2.B3 (VBUS), U2.C2 (VBUS), U2.C3 (VBUS), U2.D2 (VBUS), U2.D3 (VBUS), U2.E2 (VBUS), U2.E3 (VBUS), U2.F2 (VBUS), U2.F3 (VBUS), U2.G1 (EN0), U2.G2 (VBUS)
Changed lines of the file:
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@@
     (stroke (width 0) (type default))
   )
-  (wire (pts (xy 118.11 48.26) (xy 118.11 53.34))
-    (stroke (width 0) (type default))
-  )
   (wire (pts (xy 309.88 161.29) (xy 309.88 175.26))
     (stroke (width 0) (type default))
@@
     (stroke (width 0) (type default))
   )
+  (wire (pts (xy 137.16 160.02) (xy 118.11 160.02))
+    (stroke (width 0) (type default))
+  )
   (wire (pts (xy 369.57 119.38) (xy 382.27 119.38))
     (stroke (width 0) (type default))
@@
     (stroke (width 0) (type default))
   )
+  (wire (pts (xy 137.16 153.67) (xy 137.16 160.02))
+    (stroke (width 0) (type default))
+  )
   (wire (pts (xy 527.05 176.53) (xy 527.05 185.42))
     (stroke (width 0) (type default))
@@
     )
   )
+  (symbol (lib_id "power:VDD") (at 137.16 153.67 0) (unit 1)
+    (in_bom yes) (on_board yes) (dnp no) (fields_autoplaced)
+    (property "Reference" "#PWR05" (at 137.16 157.48 0)
+      (effects (font (size 1.27 1.27)) hide)
+    )
+    (property "Value" "VDD" (at 137.16 149.86 0)
+      (effects (font (size 1.27 1.27)))
+    )
+    (property "Footprint" "" (at 137.16 153.67 0)
+      (effects (font (size 1.27 1.27)) hide)
+    )
+    (property "Datasheet" "" (at 137.16 153.67 0)
+      (effects (font (size 1.27 1.27)) hide)
+    )
+    (pin "1")
+    (instances
+      (project "led-matrix-v2-0"
+        (path "/7b5e6152-4719-4a0e-8c49-d86181ed9746"
+          (reference "#PWR05") (unit 1)
+        )
+      )
+    )
+  )
   (symbol (lib_id "LED:WS2812B") (at 527.05 410.21 180) (unit 1)
     (in_bom yes) (on_board yes) (dnp no) (fields_autoplaced)
@@
         )
       )
-    )
-  )
-  (symbol (lib_id "power:VDD") (at 118.11 48.26 0) (unit 1)
-    (in_bom yes) (on_board yes) (dnp no) (fields_autoplaced)
-    (property "Reference" "#PWR05" (at 118.11 52.07 0)
-      (effects (font (size 1.27 1.27)) hide)
-    )
-    (property "Value" "VDD" (at 118.11 44.45 0)
-      (effects (font (size 1.27 1.27)))
-    )
-    (property "Footprint" "" (at 118.11 48.26 0)
-      (effects (font (size 1.27 1.27)) hide)
-    )
-    (property "Datasheet" "" (at 118.11 48.26 0)
-      (effects (font (size 1.27 1.27)) hide)
-    )
-    (pin "1")
-    (instances
-      (project "led-matrix-v2-0"
-        (path "/7b5e6152-4719-4a0e-8c49-d86181ed9746"
-          (reference "#PWR05") (unit 1)
-        )
-      )
